Commit message: 添加传送带和位置控制速度控制选择

File: probot_description/urdf/PROBOT_Anno/gripper.xacro (robot description, xacro)
@@ -11,5 +11,5 @@
     <!-- finger 1 -->
     <joint name="gripper_finger_joint" type="revolute">
-      <origin xyz="0 0 0" rpy="0 0 0"/>
+      <origin xyz="-0.1 0 0.05" rpy="0 0 0"/>
       <axis xyz="0 1 0"/>
       <limit effort="1.0" velocity="3.14" lower="-0.8" upper="0.5" />
@@ -44,5 +44,5 @@
     <!-- finger 2 -->
     <bioloid_F3_fixed parent="gripper_base" name="gripper_static_finger_bracket" color="${color}">
-      <origin xyz="0 0 ${-AX12_HEIGHT-F10_HEIGHT}" rpy="0 ${PI} 0" />
+      <origin xyz="-0.1 0 ${-AX12_HEIGHT-F10_HEIGHT-0.05}" rpy="0 ${PI} 0" />
     </bioloid_F3_fixed>
     <finger parent="gripper_static_finger_bracket" name="gripper_static_finger" color="${color}">

File: probot_description/urdf/PROBOT_Anno/probot_anno_with_gripper.xacro (robot description, xacro)
@@ -1,5 +1,5 @@
-<?xml version="1.0"?>
+<?xml version="1.0" ?>
 <robot name="probot_anno" xmlns:xacro="http://ros.org/wiki/xacro">
-  <xacro:property name="M_PI" value="3.1415926536"/>
+  <xacro:property name="M_PI" value="3.1415926536" />
   <xacro:include filename="$(find probot_description)/urdf/PROBOT_Anno/materials.urdf.xacro" />
   <xacro:include filename="$(find probot_description)/urdf/PROBOT_Anno/gripper.xacro" />
@@ -29,6 +29,6 @@
   <joint name="world_joint" type="fixed">
     <parent link="world" />
-    <child link = "base_link" />
-    <origin xyz="0 0 0.0315" rpy="0.0 0.0 0.0" />
+    <child link="base_link" />
+    <origin xyz="0.70 0 0.75" rpy="0.0 0.0 0.0" />
   </joint>
   <link name="link_1">
@@ -65,5 +65,5 @@
       <origin xyz="-0.010934 0.23134 0.0051509" rpy="0 0 0" />
       <mass value="0.001" />
-        <inertia ixx="1.0" ixy="0.0" ixz="0.0" iyy="1.0" iyz="0.0" izz="1.0" />
+      <inertia ixx="1.0" ixy="0.0" ixz="0.0" iyy="1.0" iyz="0.0" izz="1.0" />
     </inertial>
     <visual>
@@ -94,5 +94,5 @@
       <origin xyz="-0.010934 0.23134 0.0051509" rpy="0 0 0" />
       <mass value="0.001" />
-        <inertia ixx="1.0" ixy="0.0" ixz="0.0" iyy="1.0" iyz="0.0" izz="1.0" />
+      <inertia ixx="1.0" ixy="0.0" ixz="0.0" iyy="1.0" iyz="0.0" izz="1.0" />
     </inertial>
     <visual>
@@ -200,5 +200,5 @@
   </link>
   <joint name="joint_6" type="continuous">
-    <origin xyz="0 -0.042 0" rpy="0 0 0" />
+    <origin xyz="0 0 0" rpy="0 0 0" />
     <parent link="link_5" />
     <child link="link_6" />
@@ -206,5 +206,5 @@
     <limit lower="-3.1416" upper="3.1416" effort="100" velocity="3" />
   </joint>
-  <link name="tool0"/>
+  <link name="tool0" />
   <joint name="joint_tool0" type="fixed">
     <origin xyz="0 0 0" rpy="${M_PI/2} 0 0" />
@@ -212,6 +212,6 @@
     <child link="tool0" />
   </joint>
-   <!-- Attach the right gripper -->
-   <!-- <gripper parent="tool0" color="Green" xyz="0 0.007 0.02" rpy="0 ${-M_PI/2} ${-M_PI/2}"/> -->
+  <!-- Attach the right gripper -->
+  <gripper parent="tool0" color="Green" xyz="0 0.007 0.02" rpy="0 ${-M_PI/2} ${-M_PI/2}" />
   <!-- Transmissions for ROS Control -->
   <xacro:macro name="transmission_block" params="joint_name">
@@ -227,12 +227,30 @@
     </transmission>
   </xacro:macro>
-  <xacro:transmission_block joint_name="joint_1"/>
-  <xacro:transmission_block joint_name="joint_2"/>
-  <xacro:transmission_block joint_name="joint_3"/>
-  <xacro:transmission_block joint_name="joint_4"/>
-  <xacro:transmission_block joint_name="joint_5"/>
-  <xacro:transmission_block joint_name="joint_6"/>
-  <!-- <xacro:transmission_block joint_name="gripper_finger_joint"/> -->
-  <xacro:include filename="$(find probot_description)/urdf/PROBOT_Anno/sensors/camera.urdf.xacro"/>
+  <xacro:transmission_block joint_name="joint_1" />
+  <xacro:transmission_block joint_name="joint_2" />
+  <xacro:transmission_block joint_name="joint_3" />
+  <xacro:transmission_block joint_name="joint_4" />
+  <xacro:transmission_block joint_name="joint_5" />
+  <xacro:transmission_block joint_name="joint_6" />
+  <xacro:macro name="transmission_block2" params="joint_name">
+    <transmission name="tran2">
+      <type>transmission_interface/SimpleTransmission</type>
+      <joint name="${joint_name}">
+        <hardwareInterface>hardware_interface/PositionJointInterface</hardwareInterface>
+      </joint>
+      <actuator name="motor2">
+        <hardwareInterface>hardware_interface/PositionJointInterface</hardwareInterface>
+        <mechanicalReduction>1</mechanicalReduction>
+      </actuator>
+    </transmission>
+  </xacro:macro>
+  <xacro:transmission_block2 joint_name="joint_1" />
+  <xacro:transmission_block2 joint_name="joint_2" />
+  <xacro:transmission_block2 joint_name="joint_3" />
+  <xacro:transmission_block2 joint_name="joint_4" />
+  <xacro:transmission_block2 joint_name="joint_5" />
+  <xacro:transmission_block2 joint_name="joint_6" />
+  <xacro:transmission_block2 joint_name="gripper_finger_joint"/>
+  <xacro:include filename="$(find probot_description)/urdf/PROBOT_Anno/sensors/camera.urdf.xacro" />
   <!-- ros_control plugin -->
   <gazebo>

File: probot_description/urdf/PROBOT_Anno/sensors/camera.gazebo.xacro (robot description, xacro)
@@ -10,9 +10,9 @@
       <update_rate>30.0</update_rate>
       <camera name="head">
-        <horizontal_fov>1.3</horizontal_fov>
+        <horizontal_fov>1.8</horizontal_fov>
         <!-- <horizontal_fov>0.95</horizontal_fov> -->
         <image>
-          <width>800</width>
-          <height>800</height>
+          <width>1000</width>
+          <height>1000</height>
           <format>R8G8B8</format>
         </image>
