Commit message: 添加了机械臂随动的平移旋转、阴影与侧面的区分

File: probot_description/urdf/PROBOT_Anno/probot_anno_with_gripper.xacro (robot description, xacro)
@@ -5,4 +5,26 @@
   <xacro:include filename="$(find probot_description)/urdf/PROBOT_Anno/gripper.xacro" />
   <link name="world" />
+  <link name="base_link">
+    <inertial>
+      <origin xyz="-0.010934 0.23134 0.0051509" rpy="0 0 0" />
+      <mass value="0.01" />
+      <inertia ixx="1.0" ixy="0.0" ixz="0.0" iyy="1.0" iyz="0.0" izz="1.0" />
+    </inertial>
+    <visual>
+      <origin xyz="0.017266 0 0.0315" rpy="0 0 0" />
+      <geometry>
+        <mesh filename="package://probot_description/meshes/PROBOT_Anno/base_link.STL" />
+      </geometry>
+      <material name="">
+        <color rgba="0.79216 0.81961 0.93333 1" />
+      </material>
+    </visual>
+    <collision>
+      <origin xyz="0.017266 0 0.0315" rpy="0 0 0" />
+      <geometry>
+        <mesh filename="package://probot_description/meshes/PROBOT_Anno/base_link.STL" />
+      </geometry>
+    </collision>
+  </link>
   <joint name="world_joint" type="fixed">
     <parent link="world" />
@@ -10,26 +32,4 @@
     <origin xyz="0 0 0.0315" rpy="0.0 0.0 0.0" />
   </joint>
-  <link name="base_link">
-    <inertial>
-      <origin xyz="-0.010934 0.23134 0.0051509" rpy="0 0 0" />
-      <mass value="0.01" />
-      <inertia ixx="1.0" ixy="0.0" ixz="0.0" iyy="1.0" iyz="0.0" izz="1.0" />
-    </inertial>
-    <visual>
-      <origin xyz="0.017266 0 0.0315" rpy="0 0 0" />
-      <geometry>
-        <mesh filename="package://probot_description/meshes/PROBOT_Anno/base_link.STL" />
-      </geometry>
-      <material name="">
-        <color rgba="0.79216 0.81961 0.93333 1" />
-      </material>
-    </visual>
-    <collision>
-      <origin xyz="0.017266 0 0.0315" rpy="0 0 0" />
-      <geometry>
-        <mesh filename="package://probot_description/meshes/PROBOT_Anno/base_link.STL" />
-      </geometry>
-    </collision>
-  </link>
   <link name="link_1">
     <inertial>
@@ -199,5 +199,5 @@
     </collision>
   </link>
-  <joint name="joint_6" type="revolute">
+  <joint name="joint_6" type="continuous">
     <origin xyz="0 -0.042 0" rpy="0 0 0" />
     <parent link="link_5" />
@@ -208,10 +208,10 @@
   <link name="tool0"/>
   <joint name="joint_tool0" type="fixed">
-    <origin xyz="0 -0.013 0" rpy="${M_PI/2} 0 0" />
+    <origin xyz="0 0 0" rpy="${M_PI/2} 0 0" />
     <parent link="link_6" />
     <child link="tool0" />
   </joint>
    <!-- Attach the right gripper -->
-   <gripper parent="tool0" color="Green" xyz="0 0.015 0.02" rpy="0 ${-M_PI/2} ${-M_PI/2}"/>
+   <!-- <gripper parent="tool0" color="Green" xyz="0 0.007 0.02" rpy="0 ${-M_PI/2} ${-M_PI/2}"/> -->
   <!-- Transmissions for ROS Control -->
   <xacro:macro name="transmission_block" params="joint_name">
@@ -233,5 +233,5 @@
   <xacro:transmission_block joint_name="joint_5"/>
   <xacro:transmission_block joint_name="joint_6"/>
-  <xacro:transmission_block joint_name="gripper_finger_joint"/>
+  <!-- <xacro:transmission_block joint_name="gripper_finger_joint"/> -->
   <xacro:include filename="$(find probot_description)/urdf/PROBOT_Anno/sensors/camera.urdf.xacro"/>
   <!-- ros_control plugin -->

File: probot_description/urdf/PROBOT_Anno/sensors/camera.gazebo.xacro (robot description, xacro)
@@ -27,5 +27,5 @@
                channels, which at that point lie in the range [0,1]. -->
           <mean>0.0</mean>
-          <stddev>0.007</stddev>
+          <stddev>0.0</stddev>
         </noise>
       </camera>

File: probot_description/urdf/PROBOT_Anno/sensors/camera.urdf.xacro (robot description, xacro)
@@ -5,5 +5,5 @@
 <robot name="camera" xmlns:xacro="http://ros.org/wiki/xacro">
    <joint name="camera_joint" type="fixed">
-        <origin xyz="0 0.01 0.06" rpy="0 ${-M_PI/2} 0"/>
+        <origin xyz="0 0 0.05" rpy="0 ${-M_PI/2} 0"/>
         <parent link="tool0"/>
         <child link="camera_link"/>

Commit message: 加入深度相机与多视图几何方法计算深度信息

File: probot_description/urdf/PROBOT_Anno/probot_anno_with_gripper.xacro (robot description, xacro)
@@ -233,5 +233,5 @@
   <xacro:transmission_block joint_name="joint_5" />
   <xacro:transmission_block joint_name="joint_6" />
-  <xacro:macro name="transmission_block2" params="joint_name">
+  <!-- <xacro:macro name="transmission_block2" params="joint_name">
     <transmission name="tran2">
       <type>transmission_interface/SimpleTransmission</type>
@@ -250,6 +250,6 @@
   <xacro:transmission_block2 joint_name="joint_4" />
   <xacro:transmission_block2 joint_name="joint_5" />
-  <xacro:transmission_block2 joint_name="joint_6" />
-  <xacro:transmission_block2 joint_name="gripper_finger_joint"/>
+  <xacro:transmission_block2 joint_name="joint_6" /> -->
+  <xacro:transmission_block joint_name="gripper_finger_joint"/>
   <xacro:include filename="$(find probot_description)/urdf/PROBOT_Anno/sensors/camera.urdf.xacro" />
   <!-- ros_control plugin -->

File: probot_description/urdf/PROBOT_Anno/sensors/camera.gazebo.xacro (robot description, xacro)
@@ -7,9 +7,9 @@
   <gazebo reference="camera_link">
     <material>Gazebo/Red</material>
-    <sensor type="camera" name="camera">
+    <sensor type="depth" name="camera">
+    <!-- <sensor type="camera" name="camera"> -->
       <update_rate>30.0</update_rate>
       <camera name="head">
         <horizontal_fov>1.8</horizontal_fov>
-        <!-- <horizontal_fov>0.95</horizontal_fov> -->
         <image>
           <width>1000</width>
@@ -21,21 +21,22 @@
           <far>300</far>
         </clip>
-        <noise>
+        <!-- <noise>
           <type>gaussian</type>
-          <!-- Noise is sampled independently per pixel on each frame.
-               That pixel's noise value is added to each of its color
-               channels, which at that point lie in the range [0,1]. -->
           <mean>0.0</mean>
           <stddev>0.0</stddev>
-        </noise>
+        </noise> -->
       </camera>
-      <plugin name="camera_controller" filename="libgazebo_ros_camera.so">
+      <!-- <plugin name="camera_controller" filename="libgazebo_ros_camera.so"> -->
+        <plugin name="camera_controller" filename="libgazebo_ros_openni_kinect.so">
         <alwaysOn>true</alwaysOn>
         <updateRate>0.0</updateRate>
         <cameraName>probot_anno/camera</cameraName>
-        <imageTopicName>image_raw</imageTopicName>
-        <cameraInfoTopicName>camera_info</cameraInfoTopicName>
+        <imageTopicName>rgb/image_raw</imageTopicName>
+        <depthImageTopicName>depth/image_raw</depthImageTopicName>
+        <pointCloudTopicName>depth/points</pointCloudTopicName>
+        <cameraInfoTopicName>rgb/camera_info</cameraInfoTopicName>
+        <depthImageCameraInfoTopicName>depth/camera_info</depthImageCameraInfoTopicName>
         <frameName>camera_link</frameName>
-        <hackBaseline>0.07</hackBaseline>
+        <baseline>0.2</baseline>
         <distortionK1>0.0</distortionK1>
         <distortionK2>0.0</distortionK2>
@@ -43,4 +44,11 @@
         <distortionT1>0.0</distortionT1>
         <distortionT2>0.0</distortionT2>
+        <pointCloudCutoff>0.001</pointCloudCutoff>
+        <pointCloudCutoffMax>60.0</pointCloudCutoffMax>
+        <CxPrime>0</CxPrime>
+        <Cx>0</Cx>
+        <Cy>0</Cy>
+        <focalLength>0</focalLength>
+        <hackBaseline>0</hackBaseline>
       </plugin>
     </sensor>

Commit message: 添加小车可用键盘控制运动

File: probot_description/urdf/PROBOT_Anno/probot_anno_with_gripper.xacro (robot description, xacro)
@@ -30,5 +30,5 @@
     <parent link="world" />
     <child link="base_link" />
-    <origin xyz="0.70 0 0.75" rpy="0.0 0.0 0.0" />
+    <origin xyz="0.70 0 0.02" rpy="0.0 0.0 0.0" />
   </joint>
   <link name="link_1">
@@ -253,4 +253,5 @@
   <xacro:transmission_block joint_name="gripper_finger_joint"/>
   <xacro:include filename="$(find probot_description)/urdf/PROBOT_Anno/sensors/camera.urdf.xacro" />
+  <!-- <xacro:include filename="$(find car_model)/robots/car_model.xacro" /> -->
   <!-- ros_control plugin -->
   <gazebo>
