Commit message: 控制小车运动的同时显示图像并抓取木块

File: dancer_car/car_model/robots/car_model.xacro (robot description, xacro)
@@ -5,5 +5,5 @@
   <xacro:property name="car_a" value="0.25" />
   <xacro:property name="car_b" value="0.16" />
-  <xacro:property name="car_c" value="0.05" />
+  <xacro:property name="car_c" value="0.16" />
   <xacro:property name="wheel_mass" value="0.1" />
   <xacro:property name="wheel_lenth" value="0.02" />
@@ -615,5 +615,5 @@
       <wheelSeparation>${car_b}</wheelSeparation>
       <wheelDiameter>${wheel_radius*2}</wheelDiameter>
-      <commandTopic>cmd_vel</commandTopic>
+      <commandTopic>cmd_car</commandTopic>
       <odometryTopic>odom</odometryTopic>
       <robotBaseFrame>world_link</robotBaseFrame>
@@ -623,5 +623,5 @@
       <covariance_yaw>0.010000</covariance_yaw>
       <torque>1</torque>
-      <topicName>cmd_vel</topicName>
+      <topicName>cmd_car</topicName>
       <broadcastTF>1</broadcastTF>
     </plugin>
@@ -633,4 +633,5 @@
       <robotNamespace>/car_model</robotNamespace>
       <robotSimType>gazebo_ros_control/DefaultRobotHWSim</robotSimType>
+      <legacyModeNS>true</legacyModeNS>
     </plugin>
   </gazebo>

File: probot_description/urdf/PROBOT_Anno/probot_anno_with_gripper.xacro (robot description, xacro)
@@ -253,5 +253,4 @@
   <xacro:transmission_block joint_name="gripper_finger_joint"/>
   <xacro:include filename="$(find probot_description)/urdf/PROBOT_Anno/sensors/camera.urdf.xacro" />
-  <!-- <xacro:include filename="$(find car_model)/robots/car_model.xacro" /> -->
   <!-- ros_control plugin -->
   <gazebo>
